File: PicShift_CameraSensor_v1/PicShift_CameraSensor_v1.kicad_sch (KiCad schematic)
At the start: 0 parts

Commit message: Added symbols and footprints, added 8x8 grid schematic
Parts:
- added C1, C2, C3, C4: 0.1uF, Capacitor_SMD:C_0805_2012Metric_Pad1.18x1.45mm_HandSolder, symbol Device:C
- added J1, J2: Conn_01x11, Connector_PinHeader_1.00mm:PinHeader_1x11_P1.00mm_Vertical, symbol Connector_Generic:Conn_01x11
- added LED1, LED10, LED11, LED12, LED13, LED14, LED15, LED16, LED17, LED18, LED19, LED2, LED20, LED21, LED22, LED23, LED24, LED25, LED26, LED27, LED28, LED29, LED3, LED30, LED31, LED32, LED33, LED34, LED35, LED36, LED37, LED38, LED39, LED4, LED40, LED41, LED42, LED43, LED44, LED45, LED46, LED47, LED48, LED49, LED5, LED50, LED51, LED52, LED53, LED54, LED55, LED56, LED57, LED58, LED59, LED6, LED60, LED61, LED62, LED63, LED64, LED7, LED8, LED9: ALS-PT19, PicShift_CameraSensor:LED_77&slash_TR8_EVE, symbol PicShift_CameraSensor:ALS-PT19-315C_L177_TR8
- added U1, U2: ADG732BSUZ, PicShift_CameraSensor:SU_48_ADI, symbol PicShift_CameraSensor:ADG732BSUZ
Connections:
- new net +3.3V: C1.1, C3.1, J1.1 (Pin_1), J2.1 (Pin_1), U1.13 (VDD), U1.14 (VDD), U2.13 (VDD), U2.14 (VDD)
- new net A0COL: J1.2 (Pin_2), U1.15 (A0)
- new net A0ROW: J2.2 (Pin_2), U2.15 (A0)
- new net A1COL: J1.3 (Pin_3), U1.16 (A1)
- new net A1ROW: J2.3 (Pin_3), U2.16 (A1)
- new net A2COL: J1.4 (Pin_4), U1.17 (A2)
- new net A2ROW: J2.4 (Pin_4), U2.17 (A2)
- new net A3COL: J1.5 (Pin_5), U1.18 (A3)
- new net A3ROW: J2.5 (Pin_5), U2.18 (A3)
- new net A4COL: J1.6 (Pin_6), U1.19 (A4)
- new net A4ROW: J2.6 (Pin_6), U2.19 (A4)
- new net COL1: LED1.2, LED17.2, LED25.2, LED33.2, LED41.2, LED49.2, LED57.2, LED9.2, U1.12 (S1)
- new net COL2: LED10.2, LED18.2, LED2.2, LED26.2, LED34.2, LED42.2, LED50.2, LED58.2, U1.11 (S2)
- new net COL3: LED11.2, LED19.2, LED27.2, LED3.2, LED35.2, LED43.2, LED51.2, LED59.2, U1.10 (S3)
- new net COL4: LED12.2, LED20.2, LED28.2, LED36.2, LED4.2, LED44.2, LED52.2, LED60.2, U1.9 (S4)
- new net COL5: LED13.2, LED21.2, LED29.2, LED37.2, LED45.2, LED5.2, LED53.2, LED61.2, U1.8 (S5)
- new net COL6: LED14.2, LED22.2, LED30.2, LED38.2, LED46.2, LED54.2, LED6.2, LED62.2, U1.7 (S6)
- new net COL7: LED15.2, LED23.2, LED31.2, LED39.2, LED47.2, LED55.2, LED63.2, LED7.2, U1.6 (S7)
- new net COL8: LED16.2, LED24.2, LED32.2, LED40.2, LED48.2, LED56.2, LED64.2, LED8.2, U1.5 (S8)
- new net CSCOL: J1.7 (Pin_7), U1.20 (CS*)
- new net CSROW: J2.7 (Pin_7), U2.20 (CS*)
- new net ENCOL: J1.9 (Pin_9), U1.22 (EN*)
- new net ENROW: J2.9 (Pin_9), U2.22 (EN*)
- new net GND: C1.2, C2.2, C3.2, C4.2, J1.11 (Pin_11), J2.11 (Pin_11), U1.23 (GND), U1.24 (VSS), U2.23 (GND), U2.24 (VSS)
- new net OUTCOL: C2.1, J1.10 (Pin_10), U1.43 (D)
- new net OUTROW: C4.1, J2.10 (Pin_10), U2.43 (D)
- new net ROW1: LED1.1, LED2.1, LED3.1, LED4.1, LED5.1, LED6.1, LED7.1, LED8.1, U2.12 (S1)
- new net ROW2: LED10.1, LED11.1, LED12.1, LED13.1, LED14.1, LED15.1, LED16.1, LED9.1, U2.11 (S2)
- new net ROW3: LED17.1, LED18.1, LED19.1, LED20.1, LED21.1, LED22.1, LED23.1, LED24.1, U2.10 (S3)
- new net ROW4: LED25.1, LED26.1, LED27.1, LED28.1, LED29.1, LED30.1, LED31.1, LED32.1, U2.9 (S4)
- new net ROW5: LED33.1, LED34.1, LED35.1, LED36.1, LED37.1, LED38.1, LED39.1, LED40.1, U2.8 (S5)
- new net ROW6: LED41.1, LED42.1, LED43.1, LED44.1, LED45.1, LED46.1, LED47.1, LED48.1, U2.7 (S6)
- new net ROW7: LED49.1, LED50.1, LED51.1, LED52.1, LED53.1, LED54.1, LED55.1, LED56.1, U2.6 (S7)
- new net ROW8: LED57.1, LED58.1, LED59.1, LED60.1, LED61.1, LED62.1, LED63.1, LED64.1, U2.5 (S8)
- new net WRCOL: J1.8 (Pin_8), U1.21 (WR*)
- new net WRROW: J2.8 (Pin_8), U2.21 (WR*)
- no-connect marks 0 -> 49
Other:
- note added: "I RECEIVE COL SIGNALS!"
- note added: "I SEND ROW SIGNALS!"
- title: (none) -> Camera Sensor
